Commit message: Adicionado as constantes fisicas do mambo e adicionado o controle de atitude e posição, mas ainda falta ajustar o controle de altitude

File: rotors_description/urdf/mambo.xacro (robot description, xacro)
@@ -13,9 +13,9 @@
   <xacro:property name="rotor_offset_top" value="0" /> <!-- [m] -->
   <xacro:property name="radius_rotor" value="0.033" /> <!-- [m] -->
-  <xacro:property name="motor_constant" value="2.35e-06" /> <!-- [kg.m/s^2] -->
+  <xacro:property name="motor_constant" value="4e-06" /> <!-- [kg.m/s^2] -->
   <xacro:property name="moment_constant" value="0.016" /> <!-- [m] -->
   <xacro:property name="time_constant_up" value="0.0125" /> <!-- [s] -->
   <xacro:property name="time_constant_down" value="0.025" /> <!-- [s] -->
-  <xacro:property name="max_rot_velocity" value="320" /> <!-- [rad/s] -->
+  <xacro:property name="max_rot_velocity" value="250" /> <!-- [rad/s] -->
   <xacro:property name="sin30" value="0.5" />
   <xacro:property name="cos30" value="0.866025403784" />

Commit message: Concertado o bug das helices

File: rotors_description/urdf/mambo.xacro (robot description, xacro)
@@ -3,5 +3,5 @@
   <!-- Properties -->
   <xacro:property name="namespace" value="$(arg namespace)" />
-  <xacro:property name="rotor_velocity_slowdown_sim" value="1" />
+  <xacro:property name="rotor_velocity_slowdown_sim" value="15" />
   <xacro:property name="use_mesh_file" value="true" />
   <xacro:property name="mesh_file" value="package://rotors_description/meshes/mambo/hull.dae" />
@@ -11,5 +11,5 @@
   <xacro:property name="mass_rotor" value="0.001" /> <!-- [kg] -->
   <xacro:property name="arm_length" value="0.0425" /> <!-- [m] -->
-  <xacro:property name="rotor_offset_top" value="0" /> <!-- [m] -->
+  <xacro:property name="rotor_offset_top" value="0.01" /> <!-- [m] -->
   <xacro:property name="radius_rotor" value="0.033" /> <!-- [m] -->
   <xacro:property name="motor_constant" value="4e-06" /> <!-- [kg.m/s^2] -->
@@ -17,5 +17,5 @@
   <xacro:property name="time_constant_up" value="0.0125" /> <!-- [s] -->
   <xacro:property name="time_constant_down" value="0.025" /> <!-- [s] -->
-  <xacro:property name="max_rot_velocity" value="250" /> <!-- [rad/s] -->
+  <xacro:property name="max_rot_velocity" value="320" /> <!-- [rad/s] -->
   <xacro:property name="sin30" value="0.5" />
   <xacro:property name="cos30" value="0.866025403784" />
@@ -29,5 +29,9 @@
   <!-- inertia of a single rotor, assuming it is a cuboid. Height=3mm, width=15mm -->
   <xacro:property name="rotor_inertia">
-    <xacro:box_inertia x="${radius_rotor}" y="0.015" z="0.003" mass="${mass_rotor*rotor_velocity_slowdown_sim}" />
+    <inertia
+    ixx="${1/12 * mass_rotor * (0.031 * 0.031 + 0.005 * 0.005) * rotor_velocity_slowdown_sim}"
+    iyy="${1/12 * mass_rotor * (4 * radius_rotor * radius_rotor + 0.005 * 0.005) * rotor_velocity_slowdown_sim}"
+    izz="${1/12 * mass_rotor * (4 * radius_rotor * radius_rotor + 0.031 * 0.031) * rotor_velocity_slowdown_sim}"
+    ixy="0.0" ixz="0.0"  iyz="0.0" /> <!-- [kg*m^2] [kg*m^2] [kg*m^2] [kg*m^2] [kg*m^2] [kg*m^2] -->
   </xacro:property>
   <!-- Included URDF Files -->
@@ -63,5 +67,5 @@
     use_own_mesh="true"
     mesh="package://rotors_description/meshes/mambo/propeller_fr.dae">
-    <origin xyz="${arm_length} -${arm_length} ${rotor_offset_top}" rpy="0 0 0" />
+    <origin xyz="0.0416 -0.0425 ${rotor_offset_top}" rpy="0 0 0" />
     <xacro:insert_block name="rotor_inertia" />
   </xacro:vertical_rotor>
@@ -84,5 +88,5 @@
     use_own_mesh="true"
     mesh="package://rotors_description/meshes/mambo/propeller_rl.dae">
-    <origin xyz="-${arm_length} ${arm_length} ${rotor_offset_top}" rpy="0 0 0" />
+    <origin xyz="-0.0436 0.0425 ${rotor_offset_top}" rpy="0 0 0" />
     <xacro:insert_block name="rotor_inertia" />
   </xacro:vertical_rotor>
@@ -104,5 +108,5 @@
     use_own_mesh="true"
     mesh="package://rotors_description/meshes/mambo/propeller_fl.dae">
-    <origin xyz="${arm_length} ${arm_length} ${rotor_offset_top}" rpy="0 0 0" />
+    <origin xyz="0.0416 0.0425 ${rotor_offset_top}" rpy="0 0 0" />
     <xacro:insert_block name="rotor_inertia" />
   </xacro:vertical_rotor>
@@ -124,5 +128,5 @@
     use_own_mesh="true"
     mesh="package://rotors_description/meshes/mambo/propeller_rr.dae">
-    <origin xyz="-${arm_length} -${arm_length} ${rotor_offset_top}" rpy="0 0 0" />
+    <origin xyz="-0.0436 -0.0425 ${rotor_offset_top}" rpy="0 0 0" />
     <xacro:insert_block name="rotor_inertia" />
   </xacro:vertical_rotor>
